File: deska.brd (EAGLE design)
At the start: 100 x 80 mm, 12 parts, among them IC1 78L05Z, T1 TIP122, T2 TIP122, T3 TIP122

Commit message: verze ESP8266-01
Parts:
- removed SL1, SL2: (no value), con-amp-quick:08P
- added ESP8022-01/1, ESP8266-01/2: (no value), con-amp-quick:04P
- moved C2 43.0 mm to (17.8, 33.0)
- moved X1 37.4 mm to (45.7, 14.0)
- moved IC1 27.9 mm to (21.6, 38.1)
- moved C1 27.7 mm to (26.7, 43.2)
- moved R2 16.7 mm to (33.0, 2.54)
- moved T1 14.0 mm to (26.7, 14.0)
- moved T2 11.5 mm to (15.2, 14.0)
- moved R1 8.98 mm to (20.3, 3.81)
- moved T3 6.48 mm to (5.08, 14.0)
Connections:
- removed net +5V: C2.+, IC1.1, SL2.8
- removed net N$9: R3.1, SL2.5
- new net N$10: ESP8266-01/2.3, R3.1
- new net N$11: C2.+, ESP8022-01/1.2, ESP8022-01/1.3, ESP8022-01/1.4, IC1.1
- net GND: now also ESP8266-01/2.4; no longer SL2.7
- net N$7: now also ESP8266-01/2.1; no longer SL2.3
- net N$8: now also ESP8266-01/2.2; no longer SL2.4
Changed lines of the file:
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@@
 </autorouter>
 <elements>
-<element name="C1" library="rcl" package="E2-5" value="" x="34.29" y="69.85"/>
-<element name="C2" library="rcl" package="E2-5" value="" x="41.91" y="68.58"/>
-<element name="IC1" library="linear" package="TO92" value="78L05Z" x="35.56" y="62.23"/>
-<element name="R1" library="rcl" package="0207/10" value="" x="29.21" y="5.08"/>
-<element name="R2" library="rcl" package="0207/10" value="" x="16.51" y="5.08"/>
+<element name="C1" library="rcl" package="E2-5" value="" x="26.67" y="43.18"/>
+<element name="C2" library="rcl" package="E2-5" value="" x="17.78" y="33.02"/>
+<element name="ESP8022-01/1" library="con-amp-quick" package="04P" value="" x="12.7" y="39.37">
+<attribute name="MPN" value="" x="12.7" y="39.37" size="1.778" layer="27" display="off"/>
+<attribute name="OC_NEWARK" value="unknown" x="12.7" y="39.37" size="1.778" layer="27" display="off"/>
+<attribute name="MF" value="" x="12.7" y="39.37" size="1.778" layer="27" display="off"/>
+<attribute name="OC_FARNELL" value="unknown" x="12.7" y="39.37" size="1.778" layer="27" display="off"/>
+</element>
+<element name="ESP8266-01/2" library="con-amp-quick" package="04P" value="" x="12.7" y="43.18">
+<attribute name="MPN" value="" x="12.7" y="43.18" size="1.778" layer="27" display="off"/>
+<attribute name="OC_NEWARK" value="unknown" x="12.7" y="43.18" size="1.778" layer="27" display="off"/>
+<attribute name="MF" value="" x="12.7" y="43.18" size="1.778" layer="27" display="off"/>
+<attribute name="OC_FARNELL" value="unknown" x="12.7" y="43.18" size="1.778" layer="27" display="off"/>
+</element>
+<element name="IC1" library="linear" package="TO92" value="78L05Z" x="21.59" y="38.1"/>
+<element name="R1" library="rcl" package="0207/10" value="" x="20.32" y="3.81"/>
+<element name="R2" library="rcl" package="0207/10" value="" x="33.02" y="2.54"/>
 <element name="R3" library="rcl" package="0207/10" value="" x="7.62" y="2.54"/>
-<element name="SL1" library="con-amp-quick" package="08P" value="" x="16.51" y="57.15">
-<attribute name="MPN" value="" x="16.51" y="57.15" size="1.778" layer="27" display="off"/>
-<attribute name="OC_FARNELL" value="unknown" x="16.51" y="57.15" size="1.778" layer="27" display="off"/>
-<attribute name="MF" value="" x="16.51" y="57.15" size="1.778" layer="27" display="off"/>
-<attribute name="OC_NEWARK" value="unknown" x="16.51" y="57.15" size="1.778" layer="27" display="off"/>
-</element>
-<element name="SL2" library="con-amp-quick" package="08P" value="" x="16.51" y="71.12">
-<attribute name="MPN" value="" x="16.51" y="71.12" size="1.778" layer="27" display="off"/>
-<attribute name="OC_FARNELL" value="unknown" x="16.51" y="71.12" size="1.778" layer="27" display="off"/>
-<attribute name="MF" value="" x="16.51" y="71.12" size="1.778" layer="27" display="off"/>
-<attribute name="OC_NEWARK" value="unknown" x="16.51" y="71.12" size="1.778" layer="27" display="off"/>
-</element>
-<element name="T1" library="transistor" package="TO220" value="TIP122" x="40.64" y="15.24"/>
-<element name="T2" library="transistor" package="TO220" value="TIP122" x="26.67" y="15.24"/>
-<element name="T3" library="transistor" package="TO220" value="TIP122" x="11.43" y="15.24"/>
-<element name="X1" library="con-wago-508" package="W237-4P" value="" x="24.13" y="44.45">
-<attribute name="MPN" value="" x="24.13" y="44.45" size="1.778" layer="27" display="off"/>
-<attribute name="OC_FARNELL" value="unknown" x="24.13" y="44.45" size="1.778" layer="27" display="off"/>
-<attribute name="MF" value="" x="24.13" y="44.45" size="1.778" layer="27" display="off"/>
-<attribute name="OC_NEWARK" value="unknown" x="24.13" y="44.45" size="1.778" layer="27" display="off"/>
+<element name="T1" library="transistor" package="TO220" value="TIP122" x="26.67" y="13.97"/>
+<element name="T2" library="transistor" package="TO220" value="TIP122" x="15.24" y="13.97"/>
+<element name="T3" library="transistor" package="TO220" value="TIP122" x="5.08" y="13.97"/>
+<element name="X1" library="con-wago-508" package="W237-4P" value="" x="45.72" y="13.97">
+<attribute name="MPN" value="" x="45.72" y="13.97" size="1.778" layer="27" display="off"/>
+<attribute name="OC_NEWARK" value="unknown" x="45.72" y="13.97" size="1.778" layer="27" display="off"/>
+<attribute name="MF" value="" x="45.72" y="13.97" size="1.778" layer="27" display="off"/>
+<attribute name="OC_FARNELL" value="unknown" x="45.72" y="13.97" size="1.778" layer="27" display="off"/>
 </element>
 </elements>
@@
 <contactref element="T2" pad="3"/>
 <contactref element="T3" pad="3"/>
-<contactref element="SL2" pad="7"/>
 <contactref element="IC1" pad="2"/>
 <contactref element="C1" pad="-"/>
 <contactref element="C2" pad="-"/>
-<wire x1="29.21" y1="8.89" x2="13.97" y2="8.89" width="0" layer="19" extent="1-1"/>
-<wire x1="43.18" y1="8.89" x2="29.21" y2="8.89" width="0" layer="19" extent="1-1"/>
-<wire x1="22.86" y1="71.12" x2="43.18" y2="8.89" width="0" layer="19" extent="1-1"/>
-<wire x1="35.56" y1="64.135" x2="22.86" y2="71.12" width="0" layer="19" extent="1-1"/>
-<wire x1="35.306" y1="69.85" x2="35.56" y2="64.135" width="0" layer="19" extent="1-1"/>
-<wire x1="42.926" y1="68.58" x2="35.306" y2="69.85" width="0" layer="19" extent="1-1"/>
+<contactref element="ESP8266-01/2" pad="4"/>
+<wire x1="17.78" y1="7.62" x2="7.62" y2="7.62" width="0" layer="19" extent="1-1"/>
+<wire x1="29.21" y1="7.62" x2="17.78" y2="7.62" width="0" layer="19" extent="1-1"/>
+<wire x1="16.51" y1="43.18" x2="29.21" y2="7.62" width="0" layer="19" extent="1-1"/>
+<wire x1="21.59" y1="40.005" x2="16.51" y2="43.18" width="0" layer="19" extent="1-1"/>
+<wire x1="27.686" y1="43.18" x2="21.59" y2="40.005" width="0" layer="19" extent="1-1"/>
+<wire x1="18.796" y1="33.02" x2="27.686" y2="43.18" width="0" layer="19" extent="1-1"/>
 </signal>
 <signal name="+12V">
@@
 <contactref element="IC1" pad="3"/>
 <contactref element="C1" pad="+"/>
-<wire x1="31.75" y1="43.815" x2="36.83" y2="62.23" width="0" layer="19" extent="1-1"/>
-<wire x1="33.274" y1="69.85" x2="36.83" y2="62.23" width="0" layer="19" extent="1-1"/>
+<wire x1="25.654" y1="43.18" x2="22.86" y2="38.1" width="0" layer="19" extent="1-1"/>
+<wire x1="53.34" y1="13.335" x2="22.86" y2="38.1" width="0" layer="19" extent="1-1"/>
 </signal>
 <signal name="N$1">
 <contactref element="T1" pad="2"/>
 <contactref element="X1" pad="3"/>
-<wire x1="26.67" y1="43.815" x2="40.64" y2="8.89" width="0" layer="19" extent="1-1"/>
+<wire x1="48.26" y1="13.335" x2="26.67" y2="7.62" width="0" layer="19" extent="1-1"/>
 </signal>
 <signal name="N$2">
 <contactref element="X1" pad="2"/>
 <contactref element="T2" pad="2"/>
-<wire x1="21.59" y1="43.815" x2="26.67" y2="8.89" width="0" layer="19" extent="1-1"/>
+<wire x1="43.18" y1="13.335" x2="15.24" y2="7.62" width="0" layer="19" extent="1-1"/>
 </signal>
 <signal name="N$3">
 <contactref element="X1" pad="1"/>
 <contactref element="T3" pad="2"/>
-<wire x1="16.51" y1="43.815" x2="11.43" y2="8.89" width="0" layer="19" extent="1-1"/>
+<wire x1="38.1" y1="13.335" x2="5.08" y2="7.62" width="0" layer="19" extent="1-1"/>
 </signal>
 <signal name="N$4">
 <contactref element="T1" pad="1"/>
 <contactref element="R1" pad="2"/>
-<wire x1="38.1" y1="8.89" x2="34.29" y2="5.08" width="0" layer="19" extent="1-1"/>
+<wire x1="24.13" y1="7.62" x2="25.4" y2="3.81" width="0" layer="19" extent="1-1"/>
 </signal>
 <signal name="N$5">
 <contactref element="T2" pad="1"/>
 <contactref element="R2" pad="2"/>
-<wire x1="21.59" y1="5.08" x2="24.13" y2="8.89" width="0" layer="19" extent="1-1"/>
+<wire x1="38.1" y1="2.54" x2="12.7" y2="7.62" width="0" layer="19" extent="1-1"/>
 </signal>
 <signal name="N$6">
 <contactref element="T3" pad="1"/>
 <contactref element="R3" pad="2"/>
-<wire x1="12.7" y1="2.54" x2="8.89" y2="8.89" width="0" layer="19" extent="1-1"/>
+<wire x1="12.7" y1="2.54" x2="2.54" y2="7.62" width="0" layer="19" extent="1-1"/>
 </signal>
-<signal name="+5V">
-<contactref element="SL2" pad="8"/>
+<signal name="N$7">
+<contactref element="R1" pad="1"/>
+<contactref element="ESP8266-01/2" pad="1"/>
+<wire x1="15.24" y1="3.81" x2="8.89" y2="43.18" width="0" layer="19" extent="1-1"/>
+</signal>
+<signal name="N$8">
+<contactref element="R2" pad="1"/>
+<contactref element="ESP8266-01/2" pad="2"/>
+<wire x1="27.94" y1="2.54" x2="11.43" y2="43.18" width="0" layer="19" extent="1-1"/>
+</signal>
+<signal name="N$10">
+<contactref element="R3" pad="1"/>
+<contactref element="ESP8266-01/2" pad="3"/>
+<wire x1="13.97" y1="43.18" x2="2.54" y2="2.54" width="0" layer="19" extent="1-1"/>
+</signal>
+<signal name="N$11">
 <contactref element="IC1" pad="1"/>
 <contactref element="C2" pad="+"/>
-<wire x1="34.29" y1="62.23" x2="25.4" y2="71.12" width="0" layer="19" extent="1-1"/>
-<wire x1="40.894" y1="68.58" x2="34.29" y2="62.23" width="0" layer="19" extent="1-1"/>
-</signal>
-<signal name="N$7">
-<contactref element="SL2" pad="3"/>
-<contactref element="R1" pad="1"/>
-<wire x1="24.13" y1="5.08" x2="12.7" y2="71.12" width="0" layer="19" extent="1-1"/>
-</signal>
-<signal name="N$8">
-<contactref element="SL2" pad="4"/>
-<contactref element="R2" pad="1"/>
-<wire x1="11.43" y1="5.08" x2="15.24" y2="71.12" width="0" layer="19" extent="1-1"/>
-</signal>
-<signal name="N$9">
-<contactref element="R3" pad="1"/>
-<contactref element="SL2" pad="5"/>
-<wire x1="17.78" y1="71.12" x2="2.54" y2="2.54" width="0" layer="19" extent="1-1"/>
+<contactref element="ESP8022-01/1" pad="2"/>
+<contactref element="ESP8022-01/1" pad="3"/>
+<contactref element="ESP8022-01/1" pad="4"/>
+<wire x1="16.764" y1="33.02" x2="20.32" y2="38.1" width="0" layer="19" extent="1-1"/>
+<wire x1="13.97" y1="39.37" x2="16.764" y2="33.02" width="0" layer="19" extent="1-1"/>
+<wire x1="11.43" y1="39.37" x2="13.97" y2="39.37" width="0" layer="19" extent="1-1"/>
+<wire x1="16.51" y1="39.37" x2="13.97" y2="39.37" width="0" layer="19" extent="1-1"/>
 </signal>
 </signals>

Commit message: zmeny plosnaku
Parts:
- removed ESP8022-01/1, ESP8266-01/2: (no value), con-amp-quick:04P
- removed IC1: 78L05Z, linear:TO92
- removed X1: (no value), con-wago-508:W237-4P
- added C3: 220u, rcl:E3,5-8
- added IC2: LF33CDT, linear:TO252
- added SV1: ESP8266, con-lstb:MA04-2
- added X2: NAPAJENI, con-wago-508:W237-5P
- C1: value (none) -> 0,1u
- C2: value (none) -> 2.2u
- R1, R2, R3: value (none) -> 1k
- moved R3 49.7 mm to (11.4, 52.1), turned to 180 degrees
- moved R1 44.7 mm to (31.8, 47.0), turned to 270 degrees
- moved R2 35.8 mm to (22.9, 36.8), turned to 270 degrees
- moved C1 31.2 mm to (54.6, 57.1), turned to 270 degrees
- moved C2 30.0 mm to (35.6, 57.1), turned to 270 degrees
- moved T1 29.7 mm to (54.6, 24.1)
- moved T2 19.4 mm to (31.8, 24.1)
- moved T3 10.9 mm to (8.89, 24.1)
Connections:
- net +12V: now also IC2.1, X2.5; no longer IC1.3, X1.4
- net GND: now also C3.-, IC2.3, SV1.2, X2.1; no longer ESP8266-01/2.4, IC1.2
- net N$1: now also X2.4; no longer X1.3
- net N$10: now also SV1.4; no longer ESP8266-01/2.3
- net N$11: now also C3.+, IC2.2, SV1.3, SV1.7; no longer ESP8022-01/1.2, ESP8022-01/1.3, ESP8022-01/1.4, IC1.1
- net N$2: now also X2.3; no longer X1.2
- net N$3: now also X2.2; no longer X1.1
- net N$7: now also SV1.8; no longer ESP8266-01/2.1
- net N$8: now also SV1.6; no longer ESP8266-01/2.2
Routing:
- net GND: track 0.00 -> 199.1 mm
- net +12V: track 0.00 -> 76.1 mm
- net N$4: track 0.00 -> 44.4 mm
- net N$11: track 0.00 -> 44.2 mm
- net N$6: track 0.00 -> 39.4 mm
- net N$1: track 0.00 -> 34.9 mm
- net N$3: track 0.00 -> 28.6 mm
- net N$7: track 0.00 -> 24.1 mm
- net N$8: track 0.00 -> 20.3 mm
- net N$5: track 0.00 -> 20.3 mm
- net N$2: track 0.00 -> 10.8 mm
- net N$10: track 0.00 -> 6.35 mm
Other:
- board size 100 x 80 mm -> 64.4 x 71.1 mm

Commit message: uprava desky
Parts:
- removed C1: 0,1u, rcl:E2-5
- removed C2: 2.2u, rcl:E2-5
- removed C3: 220u, rcl:E3,5-8
- removed IC2: LF33CDT, linear:TO252
- added R4, R5, R6, R7: 10k, rcl:0207/10
- added RESET: PVA1R, switch-misc:PVA1R
- added SL1: (no value), con-amp-quick:03P
- moved R2 13.3 mm to (19.1, 49.5)
- moved R1 3.70 mm to (34.9, 48.9)
Connections:
- removed net N$11: C2.+, C3.+, IC2.2, SV1.3, SV1.7
- new net +3V3: R4.1, R5.2, R6.2, R7.1, SL1.1, SV1.3, SV1.7
- new net N$12: R7.2, RESET.2, RESET.4, SV1.5
- net +12V: now also SL1.3; no longer C1.+, IC2.1
- net GND: now also RESET.1, RESET.3, SL1.2; no longer C1.-, C2.-, C3.-, IC2.3
- net N$10: now also R6.1
- net N$7: now also R4.2
- net N$8: now also R5.1
Routing:
- net +3V3: track 0.00 -> 76.9 mm
- net N$11: track 44.2 -> 0.00 mm
- net GND: track 199.1 -> 221.5 mm
- net N$12: track 0.00 -> 22.4 mm, vias 0 -> 2
- net +12V: track 76.1 -> 55.9 mm
- net N$5: track 20.3 -> 36.8 mm
- net N$7: track 24.1 -> 35.6 mm
- net N$8: track 20.3 -> 14.0 mm
- net N$10: track 6.35 -> 11.4 mm
- net N$4: track 44.4 -> 43.2 mm

Commit message: upravy desky
Parts:
- added TX: TX, con-amp-quick:02P
- SL1: value (none) -> DCDC
- moved R1 19.6 mm to (25.4, 66.0), turned to 0 degrees
- moved R7 10.2 mm to (27.9, 59.1), turned to 270 degrees
- moved R4 1.27 mm to (11.4, 66.0)
- moved SL1 0.90 mm to (54.0, 49.5), turned to 180 degrees
- moved RESET 0.64 mm to (36.8, 63.5)
Connections:
- new net N$9: SV1.1, TX.1
- net +12V: now also X2.4; no longer X2.5
- net GND: now also TX.2
- net N$1: now also X2.5; no longer X2.4
Routing:
- net +3V3: track 76.9 -> 108.6 mm
- net N$4: track 43.2 -> 67.6 mm
- net N$7: track 35.6 -> 15.2 mm
- net N$9: track 0.00 -> 14.6 mm
- net N$1: track 34.9 -> 23.5 mm
- net GND: track 221.5 -> 211.8 mm
- net N$3: track 28.6 -> 34.9 mm
- net +12V: track 55.9 -> 57.1 mm
- net N$12: track 22.4 -> 21.7 mm, vias 2 -> 0

Commit message: deska
Parts:
- removed X2: NAPAJENI, con-wago-508:W237-5P
- added LISTA: (no value), con-wago-500:W237-6
Connections:
- net +12V: now also LISTA.4, LISTA.5; no longer X2.4
- net GND: now also LISTA.6; no longer X2.1
- net N$1: now also LISTA.3; no longer X2.5
- net N$2: now also LISTA.2; no longer X2.3
- net N$3: now also LISTA.1; no longer X2.2
Routing:
- net N$3: track 34.9 -> 18.2 mm
- net N$1: track 23.5 -> 37.7 mm
- net N$2: track 10.8 -> 15.4 mm
- net GND: track 211.8 -> 209.7 mm
Changed lines of the file:
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@@
 <element name="T2" library="transistor" package="TO220" value="TIP122" x="31.75" y="24.13"/>
 <element name="T3" library="transistor" package="TO220" value="TIP122" x="8.89" y="24.13"/>
-<element name="X2" library="con-wago-508" package="W237-5P" value="NAPAJENI" x="31.75" y="7.62">
-<attribute name="MF" value="" x="31.75" y="7.62" size="1.778" layer="27" display="off"/>
-<attribute name="MPN" value="" x="31.75" y="7.62" size="1.778" layer="27" display="off"/>
-<attribute name="OC_FARNELL" value="unknown" x="31.75" y="7.62" size="1.778" layer="27" display="off"/>
-<attribute name="OC_NEWARK" value="unknown" x="31.75" y="7.62" size="1.778" layer="27" display="off"/>
-</element>
 <element name="SV1" library="con-lstb" package="MA04-2" value="ESP8266" x="24.13" y="53.34" rot="R90">
 <attribute name="MF" value="" x="24.13" y="53.34" size="1.778" layer="27" rot="R90" display="off"/>
@@
 <attribute name="OC_NEWARK" value="unknown" x="39.37" y="51.435" size="1.778" layer="27" display="off"/>
 </element>
+<element name="LISTA" library="con-wago-500" library_urn="urn:adsk.eagle:library:195" package="W237-6" package3d_urn="urn:adsk.eagle:package:10696/1" value="" x="31.75" y="8.255">
+<attribute name="MF" value="" x="31.75" y="8.255" size="1.778" layer="27" display="off"/>
+<attribute name="MPN" value="" x="31.75" y="8.255" size="1.778" layer="27" display="off"/>
+<attribute name="OC_FARNELL" value="unknown" x="31.75" y="8.255" size="1.778" layer="27" display="off"/>
+<attribute name="OC_NEWARK" value="unknown" x="31.75" y="8.255" size="1.778" layer="27" display="off"/>
+</element>
 </elements>
 <signals>
@@
 <contactref element="T2" pad="3"/>
 <contactref element="T3" pad="3"/>
-<contactref element="X2" pad="1"/>
 <contactref element="SV1" pad="2"/>
-<wire x1="21.59" y1="13.97" x2="21.59" y2="6.985" width="1.016" layer="16"/>
-<wire x1="11.43" y1="17.78" x2="11.43" y2="13.97" width="1.016" layer="16"/>
-<wire x1="11.43" y1="13.97" x2="21.59" y2="13.97" width="1.016" layer="16"/>
 <contactref element="RESET" pad="1"/>
 <contactref element="RESET" pad="3"/>
@@
 <wire x1="40.64" y1="41.91" x2="22.86" y2="41.91" width="1.016" layer="16"/>
 <wire x1="22.86" y1="41.91" x2="22.86" y2="49.53" width="1.016" layer="16"/>
-<wire x1="57.15" y1="17.78" x2="57.15" y2="4.064" width="1.016" layer="16"/>
-<wire x1="34.29" y1="4.064" x2="57.15" y2="4.064" width="1.016" layer="16"/>
-<wire x1="34.29" y1="17.78" x2="34.29" y2="4.064" width="1.016" layer="16"/>
-<wire x1="34.29" y1="4.064" x2="29.591" y2="4.064" width="1.016" layer="16"/>
-<wire x1="29.591" y1="4.064" x2="29.21" y2="4.445" width="1.016" layer="16"/>
-<wire x1="29.21" y1="4.445" x2="29.21" y2="13.97" width="1.016" layer="16"/>
-<wire x1="29.21" y1="13.97" x2="21.59" y2="13.97" width="1.016" layer="16"/>
+<contactref element="LISTA" pad="6"/>
+<wire x1="44.25" y1="6.985" x2="44.25" y2="9.325" width="1.016" layer="16"/>
+<wire x1="44.25" y1="9.325" x2="46.355" y2="11.43" width="1.016" layer="16"/>
+<wire x1="46.355" y1="11.43" x2="54.61" y2="11.43" width="1.016" layer="16"/>
+<wire x1="54.61" y1="11.43" x2="57.15" y2="13.97" width="1.016" layer="16"/>
+<wire x1="57.15" y1="13.97" x2="57.15" y2="17.78" width="1.016" layer="16"/>
+<wire x1="42.545" y1="1.905" x2="38.735" y2="1.905" width="1.016" layer="16"/>
+<wire x1="44.25" y1="6.985" x2="44.25" y2="3.61" width="1.016" layer="16"/>
+<wire x1="44.25" y1="3.61" x2="42.545" y2="1.905" width="1.016" layer="16"/>
+<wire x1="26.035" y1="1.905" x2="27.305" y2="1.905" width="1.016" layer="16"/>
+<wire x1="36.195" y1="1.905" x2="38.735" y2="1.905" width="1.016" layer="16"/>
+<wire x1="34.29" y1="17.78" x2="34.29" y2="13.335" width="1.016" layer="16"/>
+<wire x1="31.75" y1="10.795" x2="28.575" y2="10.795" width="1.016" layer="16"/>
+<wire x1="28.575" y1="10.795" x2="26.035" y2="8.255" width="1.016" layer="16"/>
+<wire x1="26.035" y1="8.255" x2="26.035" y2="1.905" width="1.016" layer="16"/>
+<wire x1="34.29" y1="13.335" x2="31.75" y2="10.795" width="1.016" layer="16"/>
+<wire x1="11.43" y1="13.335" x2="14.605" y2="10.16" width="1.016" layer="16"/>
+<wire x1="14.605" y1="10.16" x2="20.32" y2="10.16" width="1.016" layer="16"/>
+<wire x1="20.32" y1="10.16" x2="21.59" y2="8.89" width="1.016" layer="16"/>
+<wire x1="21.59" y1="8.89" x2="21.59" y2="3.175" width="1.016" layer="16"/>
+<wire x1="21.59" y1="3.175" x2="22.86" y2="1.905" width="1.016" layer="16"/>
+<wire x1="22.86" y1="1.905" x2="26.035" y2="1.905" width="1.016" layer="16"/>
+<wire x1="11.43" y1="17.78" x2="11.43" y2="13.335" width="1.016" layer="16"/>
+<wire x1="27.305" y1="1.905" x2="36.195" y2="1.905" width="1.016" layer="16"/>
 </signal>
 <signal name="N$1">
 <contactref element="T1" pad="2"/>
-<contactref element="X2" pad="5"/>
-<wire x1="41.91" y1="6.985" x2="54.61" y2="6.985" width="1.016" layer="16"/>
-<wire x1="54.61" y1="6.985" x2="54.61" y2="17.78" width="1.016" layer="16"/>
+<contactref element="LISTA" pad="3"/>
+<wire x1="29.25" y1="6.985" x2="29.25" y2="5.675" width="1.016" layer="16"/>
+<wire x1="31.115" y1="3.81" x2="40.64" y2="3.81" width="1.016" layer="16"/>
+<wire x1="40.64" y1="3.81" x2="41.91" y2="5.08" width="1.016" layer="16"/>
+<wire x1="41.91" y1="5.08" x2="41.91" y2="9.525" width="1.016" layer="16"/>
+<wire x1="41.91" y1="9.525" x2="46.355" y2="13.97" width="1.016" layer="16"/>
+<wire x1="46.355" y1="13.97" x2="53.975" y2="13.97" width="1.016" layer="16"/>
+<wire x1="53.975" y1="13.97" x2="54.61" y2="14.605" width="1.016" layer="16"/>
+<wire x1="54.61" y1="14.605" x2="54.61" y2="17.78" width="1.016" layer="16"/>
+<wire x1="29.25" y1="5.675" x2="31.115" y2="3.81" width="1.016" layer="16"/>
 </signal>
 <signal name="N$2">
 <contactref element="T2" pad="2"/>
-<contactref element="X2" pad="3"/>
-<wire x1="31.75" y1="17.78" x2="31.75" y2="6.985" width="1.016" layer="16"/>
+<contactref element="LISTA" pad="2"/>
+<wire x1="24.25" y1="6.985" x2="24.25" y2="9.645" width="1.016" layer="16"/>
+<wire x1="27.94" y1="13.335" x2="30.48" y2="13.335" width="1.016" layer="16"/>
+<wire x1="30.48" y1="13.335" x2="31.75" y2="14.605" width="1.016" layer="16"/>
+<wire x1="31.75" y1="14.605" x2="31.75" y2="17.78" width="1.016" layer="16"/>
+<wire x1="24.25" y1="9.645" x2="27.94" y2="13.335" width="1.016" layer="16"/>
 </signal>
 <signal name="N$3">
 <contactref element="T3" pad="2"/>
-<contactref element="X2" pad="2"/>
-<wire x1="8.89" y1="17.78" x2="8.89" y2="3.81" width="1.016" layer="16"/>
-<wire x1="8.89" y1="3.81" x2="26.67" y2="3.81" width="1.016" layer="16"/>
-<wire x1="26.67" y1="3.81" x2="26.67" y2="6.985" width="1.016" layer="16"/>
+<contactref element="LISTA" pad="1"/>
+<wire x1="8.89" y1="17.78" x2="8.89" y2="12.065" width="1.016" layer="16"/>
+<wire x1="8.89" y1="12.065" x2="13.97" y2="6.985" width="1.016" layer="16"/>
+<wire x1="13.97" y1="6.985" x2="19.25" y2="6.985" width="1.016" layer="16"/>
 </signal>
 <signal name="N$4">
@@
 </signal>
 <signal name="+12V">
-<contactref element="X2" pad="4"/>
 <contactref element="SL1" pad="3"/>
 <wire x1="51.435" y1="49.53" x2="44.45" y2="49.53" width="1.016" layer="16"/>
-<wire x1="44.45" y1="49.53" x2="44.45" y2="12.7" width="1.016" layer="16"/>
-<wire x1="44.45" y1="12.7" x2="36.83" y2="12.7" width="1.016" layer="16"/>
-<wire x1="36.83" y1="12.7" x2="36.83" y2="6.985" width="1.016" layer="16"/>
+<wire x1="44.45" y1="49.53" x2="44.45" y2="15.875" width="1.016" layer="16"/>
+<contactref element="LISTA" pad="5"/>
+<wire x1="39.25" y1="6.985" x2="39.37" y2="7.105" width="1.016" layer="16"/>
+<wire x1="39.37" y1="7.105" x2="39.37" y2="10.16" width="1.016" layer="16"/>
+<wire x1="39.37" y1="10.16" x2="44.45" y2="15.24" width="1.016" layer="16"/>
+<wire x1="44.45" y1="15.24" x2="44.45" y2="15.875" width="1.016" layer="16"/>
+<contactref element="LISTA" pad="4"/>
+<wire x1="34.25" y1="6.985" x2="39.25" y2="6.985" width="1.016" layer="16"/>
 </signal>
 </signals>
