File: deska.brd (EAGLE design)
At the start: 64.4 x 71.1 mm, 15 parts, among them T1 TIP122, T2 TIP122, T3 TIP122

Commit message: deska
Parts:
- removed TX: TX, con-amp-quick:02P
- added SERIAL: (no value), con-amp-quick:03P
Connections:
- net GND: now also SERIAL.1; no longer TX.2
- net N$7: now also SERIAL.3
- net N$9: now also SERIAL.2; no longer TX.1
Routing:
- net N$7: track 15.2 -> 32.9 mm
- net GND: track 209.7 -> 197.9 mm
- net N$9: track 14.6 -> 9.52 mm
Changed lines of the file:
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@@
 <attribute name="OC_NEWARK" value="unknown" x="53.975" y="49.53" size="1.778" layer="27" rot="R180" display="off"/>
-</element>
-<element name="TX" library="con-amp-quick" library_urn="urn:adsk.eagle:library:125" package="02P" package3d_urn="urn:adsk.eagle:package:5956/1" value="TX" x="39.37" y="51.435">
-<attribute name="MF" value="" x="39.37" y="51.435" size="1.778" layer="27" display="off"/>
-<attribute name="MPN" value="" x="39.37" y="51.435" size="1.778" layer="27" display="off"/>
-<attribute name="OC_FARNELL" value="unknown" x="39.37" y="51.435" size="1.778" layer="27" display="off"/>
-<attribute name="OC_NEWARK" value="unknown" x="39.37" y="51.435" size="1.778" layer="27" display="off"/>
 </element>
 <element name="LISTA" library="con-wago-500" library_urn="urn:adsk.eagle:library:195" package="W237-6" package3d_urn="urn:adsk.eagle:package:10696/1" value="" x="31.75" y="8.255">
@@
 <attribute name="OC_FARNELL" value="unknown" x="31.75" y="8.255" size="1.778" layer="27" display="off"/>
 <attribute name="OC_NEWARK" value="unknown" x="31.75" y="8.255" size="1.778" layer="27" display="off"/>
+</element>
+<element name="SERIAL" library="con-amp-quick" library_urn="urn:adsk.eagle:library:125" package="03P" package3d_urn="urn:adsk.eagle:package:5957/1" value="" x="34.925" y="49.53" rot="R90">
+<attribute name="MF" value="" x="34.925" y="49.53" size="1.778" layer="27" rot="R90" display="off"/>
+<attribute name="MPN" value="" x="34.925" y="49.53" size="1.778" layer="27" rot="R90" display="off"/>
+<attribute name="OC_FARNELL" value="unknown" x="34.925" y="49.53" size="1.778" layer="27" rot="R90" display="off"/>
+<attribute name="OC_NEWARK" value="unknown" x="34.925" y="49.53" size="1.778" layer="27" rot="R90" display="off"/>
 </element>
 </elements>
@@
 <wire x1="39.3192" y1="66.4972" x2="39.3192" y2="60.5028" width="1.016" layer="16"/>
 <contactref element="SL1" pad="2"/>
-<wire x1="39.3192" y1="60.5028" x2="40.64" y2="60.5028" width="1.016" layer="16"/>
-<wire x1="40.64" y1="60.5028" x2="53.975" y2="60.5028" width="1.016" layer="16"/>
-<wire x1="53.975" y1="60.5028" x2="53.975" y2="49.53" width="1.016" layer="16"/>
-<contactref element="TX" pad="2"/>
+<wire x1="39.3192" y1="52.2478" x2="48.895" y2="52.2478" width="1.016" layer="16"/>
+<wire x1="48.895" y1="52.2478" x2="53.975" y2="52.2478" width="1.016" layer="16"/>
+<wire x1="53.975" y1="52.2478" x2="53.975" y2="49.53" width="1.016" layer="16"/>
 <wire x1="57.15" y1="17.78" x2="60.96" y2="17.78" width="1.016" layer="16"/>
-<wire x1="60.96" y1="40.005" x2="53.975" y2="40.005" width="1.016" layer="16"/>
-<wire x1="53.975" y1="40.005" x2="53.975" y2="49.53" width="1.016" layer="16"/>
-<wire x1="60.96" y1="17.78" x2="60.96" y2="40.005" width="1.016" layer="16"/>
-<wire x1="40.64" y1="51.435" x2="40.64" y2="60.5028" width="1.016" layer="16"/>
-<wire x1="40.64" y1="51.435" x2="40.64" y2="41.91" width="1.016" layer="16"/>
-<wire x1="40.64" y1="41.91" x2="22.86" y2="41.91" width="1.016" layer="16"/>
-<wire x1="22.86" y1="41.91" x2="22.86" y2="49.53" width="1.016" layer="16"/>
+<wire x1="60.96" y1="45.72" x2="53.975" y2="45.72" width="1.016" layer="16"/>
+<wire x1="53.975" y1="45.72" x2="53.975" y2="49.53" width="1.016" layer="16"/>
+<wire x1="60.96" y1="17.78" x2="60.96" y2="45.72" width="1.016" layer="16"/>
+<wire x1="22.86" y1="46.99" x2="34.925" y2="46.99" width="1.016" layer="16"/>
+<wire x1="22.86" y1="46.99" x2="22.86" y2="49.53" width="1.016" layer="16"/>
 <contactref element="LISTA" pad="6"/>
 <wire x1="44.25" y1="6.985" x2="44.25" y2="9.325" width="1.016" layer="16"/>
@@
 <wire x1="11.43" y1="17.78" x2="11.43" y2="13.335" width="1.016" layer="16"/>
 <wire x1="27.305" y1="1.905" x2="36.195" y2="1.905" width="1.016" layer="16"/>
+<contactref element="SERIAL" pad="1"/>
+<wire x1="34.925" y1="46.99" x2="38.735" y2="46.99" width="1.016" layer="16"/>
+<wire x1="38.735" y1="46.99" x2="39.37" y2="47.625" width="1.016" layer="16"/>
+<wire x1="39.37" y1="47.625" x2="39.37" y2="60.452" width="1.016" layer="16"/>
+<wire x1="39.37" y1="60.452" x2="39.3192" y2="60.5028" width="1.016" layer="16"/>
+<wire x1="39.3192" y1="60.5028" x2="39.3192" y2="52.2478" width="1.016" layer="16"/>
 </signal>
 <signal name="N$1">
@@
 <wire x1="22.86" y1="66.04" x2="20.32" y2="66.04" width="1.016" layer="16"/>
 <wire x1="20.32" y1="66.04" x2="16.51" y2="66.04" width="1.016" layer="16"/>
+<contactref element="SERIAL" pad="3"/>
+<wire x1="34.925" y1="52.07" x2="32.385" y2="52.07" width="1.016" layer="16"/>
+<wire x1="32.385" y1="52.07" x2="31.75" y2="51.435" width="1.016" layer="16"/>
+<wire x1="31.75" y1="51.435" x2="31.2674" y2="50.9524" width="0.3048" layer="16"/>
+<wire x1="24.13" y1="55.88" x2="22.86" y2="57.15" width="0.3048" layer="16"/>
+<wire x1="31.2674" y1="50.9524" x2="24.6126" y2="50.9524" width="0.3048" layer="16"/>
+<wire x1="24.6126" y1="50.9524" x2="24.13" y2="51.435" width="0.3048" layer="16"/>
+<wire x1="24.13" y1="51.435" x2="24.13" y2="55.88" width="0.3048" layer="16"/>
 </signal>
 <signal name="N$8">
@@
 <wire x1="27.94" y1="64.135" x2="25.4" y2="64.135" width="1.016" layer="16"/>
 </signal>
-<signal name="N$9">
-<contactref element="SV1" pad="1"/>
-<contactref element="TX" pad="1"/>
-<wire x1="25.4" y1="49.53" x2="38.1" y2="49.53" width="1.016" layer="16"/>
-<wire x1="38.1" y1="49.53" x2="38.1" y2="51.435" width="1.016" layer="16"/>
-</signal>
 <signal name="+12V">
 <contactref element="SL1" pad="3"/>
@@
 <wire x1="34.25" y1="6.985" x2="39.25" y2="6.985" width="1.016" layer="16"/>
 </signal>
+<signal name="N$9">
+<contactref element="SV1" pad="1"/>
+<contactref element="SERIAL" pad="2"/>
+<wire x1="25.4" y1="49.53" x2="32.385" y2="49.53" width="1.016" layer="16"/>
+<wire x1="32.385" y1="49.53" x2="34.925" y2="49.53" width="1.016" layer="16"/>
+</signal>
 </signals>

Commit message: zmena odporu
Parts:
- R4, R5, R6: value 10k -> 1k
Changed lines of the file:
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@@
 <attribute name="OC_NEWARK" value="unknown" x="24.13" y="53.34" size="1.778" layer="27" rot="R90" display="off"/>
 </element>
-<element name="R4" library="rcl" package="0207/10" value="10k" x="11.43" y="66.04"/>
-<element name="R5" library="rcl" package="0207/10" value="10k" x="11.43" y="62.23" rot="R180"/>
-<element name="R6" library="rcl" package="0207/10" value="10k" x="11.43" y="57.15" rot="R180"/>
+<element name="R4" library="rcl" package="0207/10" value="1k" x="11.43" y="66.04"/>
+<element name="R5" library="rcl" package="0207/10" value="1k" x="11.43" y="62.23" rot="R180"/>
+<element name="R6" library="rcl" package="0207/10" value="1k" x="11.43" y="57.15" rot="R180"/>
 <element name="R7" library="rcl" package="0207/10" value="10k" x="27.94" y="59.055" rot="R270"/>
 <element name="RESET" library="switch-misc" library_urn="urn:adsk.eagle:library:376" package="PVA1R" package3d_urn="urn:adsk.eagle:package:27429/1" value="PVA1R" x="36.83" y="63.5" rot="R270"/>

Commit message: upravy desku - popisky
Connections:
- net N$10 renamed GPIO2
- net N$12 renamed RST
- net N$7 renamed RX
- net N$8 renamed GPIO0
- net N$9 renamed TX
Changed lines of the file:
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@@
 <contactref element="SERIAL" pad="1"/>
 <wire x1="34.925" y1="46.99" x2="38.735" y2="46.99" width="1.016" layer="16"/>
-<wire x1="38.735" y1="46.99" x2="39.37" y2="47.625" width="1.016" layer="16"/>
+<wire x1="39.37" y1="47.625" x2="38.735" y2="46.99" width="1.016" layer="16"/>
 <wire x1="39.37" y1="47.625" x2="39.37" y2="60.452" width="1.016" layer="16"/>
 <wire x1="39.37" y1="60.452" x2="39.3192" y2="60.5028" width="1.016" layer="16"/>
@@
 <wire x1="3.81" y1="17.78" x2="6.35" y2="17.78" width="1.016" layer="16"/>
 </signal>
-<signal name="N$7">
+<signal name="RX">
 <contactref element="R1" pad="1"/>
 <contactref element="SV1" pad="8"/>
@@
 <wire x1="24.13" y1="51.435" x2="24.13" y2="55.88" width="0.3048" layer="16"/>
 </signal>
-<signal name="N$8">
+<signal name="GPIO0">
 <contactref element="R2" pad="1"/>
 <contactref element="SV1" pad="6"/>
@@
 <wire x1="19.05" y1="62.23" x2="16.51" y2="62.23" width="1.016" layer="16"/>
 </signal>
-<signal name="N$10">
+<signal name="GPIO2">
 <contactref element="R3" pad="1"/>
 <contactref element="SV1" pad="4"/>
@@
 <wire x1="16.51" y1="57.15" x2="16.51" y2="52.07" width="1.016" layer="16"/>
 </signal>
-<signal name="N$12">
+<signal name="RST">
 <contactref element="RESET" pad="2"/>
 <contactref element="RESET" pad="4"/>
@@
 <wire x1="34.25" y1="6.985" x2="39.25" y2="6.985" width="1.016" layer="16"/>
 </signal>
-<signal name="N$9">
+<signal name="TX">
 <contactref element="SV1" pad="1"/>
 <contactref element="SERIAL" pad="2"/>
