File: deska.brd (EAGLE design)
At the start: 64.4 x 71.1 mm, 15 parts, among them T1 TIP122, T2 TIP122, T3 TIP122

Commit message: +
Parts:
- moved R1 6.63 mm to (23.5, 59.7)
- moved R4 6.63 mm to (9.53, 59.7)
- moved R2 6.63 mm to (17.1, 43.2)
- moved R7 6.63 mm to (26.0, 52.7)
- moved RESET 6.63 mm to (34.9, 57.1)
- moved SL1 6.63 mm to (52.1, 43.2)
- moved R3 6.63 mm to (9.53, 45.7)
- moved R6 6.63 mm to (9.53, 50.8)
- moved SERIAL 6.63 mm to (33.0, 43.2)
- moved SV1 6.63 mm to (22.2, 47.0)
- moved R5 6.63 mm to (9.53, 55.9)
- moved T1 2.29 mm to (52.7, 22.9)
- moved T2 2.29 mm to (29.8, 22.9)
- moved LISTA 1.91 mm to (29.8, 8.26)
- moved T3 1.80 mm to (7.62, 22.9)
Routing:
- net GND: track 197.9 -> 180.6 mm
- net +12V: track 56.7 -> 50.3 mm
- net N$4: track 67.6 -> 62.5 mm
- net N$5: track 36.8 -> 31.8 mm
- net N$6: track 39.4 -> 34.9 mm
- net N$3: track 18.2 -> 16.6 mm
- net N$1: track 37.7 -> 36.4 mm
- net N$2: track 15.4 -> 14.1 mm
Other:
- board size 64.4 x 71.1 mm -> 60.6 x 64.1 mm
